File: hardware/Pi_Observer_board/Pi_Observer_board_schematic.sch (EAGLE design)
At the start: 17 parts, among them Q1 BC548B, U1 DS18B20, U2 DS18B20, X1 RASPI_GPIO_B+#_PIN

Commit message: Advance board and chnage gpio pins
Parts:
- JP1: value (none) -> RTC
- LED1: value (none) -> RED
- LED2: value (none) -> GREEN
- R1: value (none) -> 180
- R2, R6: value (none) -> 150
- R3: value (none) -> 1k
- R4, R5: value (none) -> 4k7
- SV2: value (none) -> HUMIDITY
- SV3: value (none) -> PRESSURE
Connections:
- removed net GPIO20: R6.1, X1.GPIO20
- removed net GPIO21: R3.1, X1.GPIO21
- new net GPIO22: R3.1, X1.GPIO22
- new net GPIO27: R6.1, X1.GPIO27
Other:
- note added: "Maciej Ziaja"
- note added: "https://github.com/MaciejZj/Pi-Observer"
- moved on the sheet: SV1
