File: hardware/Pi_Observer/Pi_Observer.sch (EAGLE design)
At the start: 17 parts, among them Q1 BC548B, U1 DS18B20, U2 DS18B20, X1 RASPI_GPIO_B+#_PIN

Commit message: Add paper sheet size on frame
Other:
- note added: "A5"
Changed lines of the file:
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@@
 universal data logger and remote
 accesss project.</text>
+<text x="172.72" y="5.08" size="2.1844" layer="94">A5</text>
 </plain>
 <instances>
